Commit message: fix: multiple color w/ paths

File: open_manipulator_x_description/urdf/open_manipulator_x.urdf.xacro (robot description, xacro)
@@ -1,10 +1,11 @@
 <?xml version="1.0"?>
-<robot name="open_manipulator_x" xmlns:xacro="http://ros.org/wiki/xacro">
-  <material name="grey">
+<robot name="open_manipulator_x"
+  xmlns:xacro="http://ros.org/wiki/xacro">
+  <!-- <material name="grey">
     <color rgba="0.5 0.5 0.5 1.0"/>
-  </material>
-  <material name="red">
+  </material> -->
+  <!-- <material name="red">
     <color rgba="0.8 0.0 0.0 1.0"/>
-  </material>
+  </material> -->
   <!-- Link 1 -->
   <link name="link1">
@@ -25,7 +26,5 @@
       <origin xyz="3.0876154e-04 0.0000000e+00 -1.2176461e-04" />
       <mass value="7.9119962e-02" />
-      <inertia ixx="1.2505234e-05" ixy="0.0" ixz="-1.7855208e-07"
-               iyy="2.1898364e-05" iyz="0.0"
-               izz="1.9267361e-05" />
+      <inertia ixx="1.2505234e-05" ixy="0.0" ixz="-1.7855208e-07" iyy="2.1898364e-05" iyz="0.0" izz="1.9267361e-05" />
     </inertial>
   </link>
@@ -53,10 +52,8 @@
       </geometry>
     </collision>
-     <inertial>
+    <inertial>
       <origin xyz="-3.0184870e-04 5.4043684e-04 0.047433464e-02" />
       <mass value="9.8406837e-02" />
-      <inertia ixx="3.4543422e-05" ixy="-1.6031095e-08" ixz="-3.8375155e-07"
-               iyy="3.2689329e-05" iyz="2.8511935e-08"
-               izz="1.8850320e-05" />
+      <inertia ixx="3.4543422e-05" ixy="-1.6031095e-08" ixz="-3.8375155e-07" iyy="3.2689329e-05" iyz="2.8511935e-08" izz="1.8850320e-05" />
     </inertial>
   </link>
@@ -87,7 +84,5 @@
       <origin xyz="1.0308393e-02 3.7743363e-04 1.0170197e-01" />
       <mass value="1.3850917e-01" />
-      <inertia ixx="3.3055381e-04" ixy="-9.7940978e-08" ixz="-3.8505711e-05"
-               iyy="3.4290447e-04" iyz="-1.5717516e-06"
-               izz="6.0346498e-05" />
+      <inertia ixx="3.3055381e-04" ixy="-9.7940978e-08" ixz="-3.8505711e-05" iyy="3.4290447e-04" iyz="-1.5717516e-06" izz="6.0346498e-05" />
     </inertial>
   </link>
@@ -115,10 +110,8 @@
       </geometry>
     </collision>
-     <inertial>
+    <inertial>
       <origin xyz="9.0909590e-02 3.8929816e-04 2.2413279e-04" />
       <mass value="1.3274562e-01" />
-      <inertia ixx="3.0654178e-05" ixy="-1.2764155e-06" ixz="-2.6874417e-07"
-               iyy="2.4230292e-04" iyz="1.1559550e-08"
-               izz="2.5155057e-04" />
+      <inertia ixx="3.0654178e-05" ixy="-1.2764155e-06" ixz="-2.6874417e-07" iyy="2.4230292e-04" iyz="1.1559550e-08" izz="2.5155057e-04" />
     </inertial>
   </link>
@@ -146,10 +139,8 @@
       </geometry>
     </collision>
-     <inertial>
+    <inertial>
       <origin xyz="4.4206755e-02 3.6839985e-07 8.9142216e-03" />
       <mass value="1.4327573e-01" />
-      <inertia ixx="8.0870749e-05" ixy="0.0" ixz="-1.0157896e-06"
-               iyy="7.5980465e-05" iyz="0.0"
-               izz="9.3127351e-05" />
+      <inertia ixx="8.0870749e-05" ixy="0.0" ixz="-1.0157896e-06" iyy="7.5980465e-05" iyz="0.0" izz="9.3127351e-05" />
     </inertial>
   </link>
@@ -180,7 +171,5 @@
       <origin xyz="0 0 0" />
       <mass value="1.0e-03" />
-      <inertia ixx="1.0e-03" ixy="0.0" ixz="0.0"
-               iyy="1.0e-03" iyz="0.0"
-               izz="1.0e-03" />
+      <inertia ixx="1.0e-03" ixy="0.0" ixz="0.0" iyy="1.0e-03" iyz="0.0" izz="1.0e-03" />
     </inertial>
   </link>
@@ -212,7 +201,5 @@
       <origin xyz="0 0 0" />
       <mass value="1.0e-03" />
-      <inertia ixx="1.0e-03" ixy="0.0" ixz="0.0"
-               iyy="1.0e-03" iyz="0.0"
-               izz="1.0e-03" />
+      <inertia ixx="1.0e-03" ixy="0.0" ixz="0.0" iyy="1.0e-03" iyz="0.0" izz="1.0e-03" />
     </inertial>
   </link>
@@ -231,11 +218,9 @@
       </geometry>
       <material name="red"/>
-     </visual>
+    </visual>
     <inertial>
       <origin xyz="0 0 0" />
       <mass value="1.0e-03" />
-      <inertia ixx="1.0e-03" ixy="0.0" ixz="0.0"
-               iyy="1.0e-03" iyz="0.0"
-               izz="1.0e-03" />
+      <inertia ixx="1.0e-03" ixy="0.0" ixz="0.0" iyy="1.0e-03" iyz="0.0" izz="1.0e-03" />
     </inertial>
   </link>

File: open_manipulator_x_description/urdf/open_manipulator_x_robot.urdf.xacro (robot description, xacro)
@@ -1,15 +1,16 @@
 <?xml version="1.0"?>
 <!-- OpenManipulator Chain -->
-<robot name="open_manipulator_x" xmlns:xacro="http://ros.org/wiki/xacro">
+<robot name="open_manipulator_x"
+  xmlns:xacro="http://ros.org/wiki/xacro">
   <!-- Import Rviz colors -->
-  <xacro:include filename="package://open_manipulator_x_description/urdf/materials.xacro" />
+  <xacro:include filename="$(find open_manipulator_x_description)/urdf/materials.xacro" />
   <!-- Import all Gazebo-customization elements, including Gazebo colors -->
   <xacro:if value="$(arg gazebo)">
-    <xacro:include filename="package://open_manipulator_x_description/urdf/open_manipulator_x.gazebo.xacro" />
+    <xacro:include filename="$(find open_manipulator_x_description)/urdf/open_manipulator_x.gazebo.xacro" />
   </xacro:if>
   <!-- Import Transmission -->
-  <xacro:include filename="package://open_manipulator_x_description/urdf/open_manipulator_x.transmission.xacro" />
+  <xacro:include filename="$(find open_manipulator_x_description)/urdf/open_manipulator_x.transmission.xacro" />
   <!-- Import URDF -->
-  <xacro:include filename="package://open_manipulator_x_description/urdf/open_manipulator_x.urdf.xacro" />
+  <xacro:include filename="$(find open_manipulator_x_description)/urdf/open_manipulator_x.urdf.xacro" />
   <!-- World -->
   <link name="world"/>
@@ -23,8 +24,8 @@
   <!-- TODO:Xacro files do not work yet -->
   <!-- !!!!!!!!!!!!!!!!!!!!!!!!!!!!!!!! -->
-  <material name="black">
+  <!-- <material name="black">
     <color rgba="0.0 0.0 0.0 1.0"/>
-  </material>
-  <material name="white">
+  </material> -->
+  <!-- <material name="white">
     <color rgba="1.0 1.0 1.0 1.0"/>
   </material>
@@ -37,21 +38,21 @@
   <material name="green">
     <color rgba="0.0 0.8 0.0 1.0"/>
-  </material>
-  <material name="grey">
+  </material> -->
+  <!-- <material name="grey">
     <color rgba="0.5 0.5 0.5 1.0"/>
-  </material>
+  </material> -->
   <!-- Link 1 -->
-  <link name="link1">
-    <visual>
-      <origin xyz="0 0 0" rpy="0 0 0"/>
-      <geometry>
-        <mesh filename="package://open_manipulator_x_description/meshes/chain_link1.stl" scale="0.001 0.001 0.001"/>
-      </geometry>
-      <material name="grey"/>
-    </visual>
-    <collision>
-      <origin xyz="0 0 0" rpy="0 0 0"/>
-      <geometry>
-        <mesh filename="package://open_manipulator_x_description/meshes/chain_link1.stl" scale="0.001 0.001 0.001"/>
+  <!-- <link name="link1">
+    <visual>
+      <origin xyz="0 0 0" rpy="0 0 0"/>
+      <geometry>
+        <mesh filename="file://$(find open_manipulator_x_description)/meshes/chain_link1.stl" scale="0.001 0.001 0.001"/>
+      </geometry>
+      <material name="grey"/>
+    </visual>
+    <collision>
+      <origin xyz="0 0 0" rpy="0 0 0"/>
+      <geometry>
+        <mesh filename="file://$(find open_manipulator_x_description)/meshes/chain_link1.stl" scale="0.001 0.001 0.001"/>
       </geometry>
     </collision>
@@ -59,11 +60,9 @@
       <origin xyz="3.0876154e-04 0.0000000e+00 -1.2176461e-04" />
       <mass value="7.9119962e-02" />
-      <inertia ixx="1.2505234e-05" ixy="0.0" ixz="-1.7855208e-07"
-               iyy="2.1898364e-05" iyz="0.0"
-               izz="1.9267361e-05" />
-    </inertial>
-  </link>
+      <inertia ixx="1.2505234e-05" ixy="0.0" ixz="-1.7855208e-07" iyy="2.1898364e-05" iyz="0.0" izz="1.9267361e-05" />
+    </inertial>
+  </link> -->
   <!-- Joint 1 -->
-  <joint name="joint1" type="revolute">
+  <!-- <joint name="joint1" type="revolute">
     <parent link="link1"/>
     <child link="link2"/>
@@ -71,11 +70,11 @@
     <axis xyz="0 0 1"/>
     <limit velocity="4.8" effort="1" lower="-2.82743338823" upper="2.82743338823" />
-  </joint>
+  </joint> -->
   <!--  Link 2 -->
-  <link name="link2">
+  <!-- <link name="link2">
     <visual>
       <origin xyz="0 0 0.019" rpy="0 0 0"/>
       <geometry>
-        <mesh filename="package://open_manipulator_x_description/meshes/chain_link2.stl" scale="0.001 0.001 0.001"/>
+        <mesh filename="file://$(find open_manipulator_x_description)/meshes/chain_link2.stl" scale="0.001 0.001 0.001"/>
       </geometry>
       <material name="grey"/>
@@ -84,17 +83,15 @@
       <origin xyz="0 0 0.019" rpy="0 0 0"/>
       <geometry>
-        <mesh filename="package://open_manipulator_x_description/meshes/chain_link2.stl" scale="0.001 0.001 0.001"/>
-      </geometry>
-    </collision>
-     <inertial>
+        <mesh filename="file://$(find open_manipulator_x_description)/meshes/chain_link2.stl" scale="0.001 0.001 0.001"/>
+      </geometry>
+    </collision>
+    <inertial>
       <origin xyz="-3.0184870e-04 5.4043684e-04 0.047433464e-02" />
       <mass value="9.8406837e-02" />
-      <inertia ixx="3.4543422e-05" ixy="-1.6031095e-08" ixz="-3.8375155e-07"
-               iyy="3.2689329e-05" iyz="2.8511935e-08"
-               izz="1.8850320e-05" />
-    </inertial>
-  </link>
+      <inertia ixx="3.4543422e-05" ixy="-1.6031095e-08" ixz="-3.8375155e-07" iyy="3.2689329e-05" iyz="2.8511935e-08" izz="1.8850320e-05" />
+    </inertial>
+  </link> -->
   <!--  Joint 2 -->
-  <joint name="joint2" type="revolute">
+  <!-- <joint name="joint2" type="revolute">
     <parent link="link2"/>
     <child link="link3"/>
@@ -102,18 +99,18 @@
     <axis xyz="0 1 0"/>
     <limit velocity="4.8" effort="1" lower="-1.79070781255" upper="1.57079632679" />
-  </joint>
+  </joint> -->
   <!--  Link 3 -->
-  <link name="link3">
-    <visual>
-      <origin xyz="0 0 0" rpy="0 0 0"/>
-      <geometry>
-        <mesh filename="package://open_manipulator_x_description/meshes/chain_link3.stl" scale="0.001 0.001 0.001"/>
-      </geometry>
-      <material name="grey"/>
-    </visual>
-    <collision>
-      <origin xyz="0 0 0" rpy="0 0 0"/>
-      <geometry>
-        <mesh filename="package://open_manipulator_x_description/meshes/chain_link3.stl" scale="0.001 0.001 0.001"/>
+  <!-- <link name="link3">
+    <visual>
+      <origin xyz="0 0 0" rpy="0 0 0"/>
+      <geometry>
+        <mesh filename="file://$(find open_manipulator_x_description)/meshes/chain_link3.stl" scale="0.001 0.001 0.001"/>
+      </geometry>
+      <material name="grey"/>
+    </visual>
+    <collision>
+      <origin xyz="0 0 0" rpy="0 0 0"/>
+      <geometry>
+        <mesh filename="file://$(find open_manipulator_x_description)/meshes/chain_link3.stl" scale="0.001 0.001 0.001"/>
       </geometry>
     </collision>
@@ -121,11 +118,9 @@
       <origin xyz="1.0308393e-02 3.7743363e-04 1.0170197e-01" />
       <mass value="1.3850917e-01" />
-      <inertia ixx="3.3055381e-04" ixy="-9.7940978e-08" ixz="-3.8505711e-05"
-               iyy="3.4290447e-04" iyz="-1.5717516e-06"
-               izz="6.0346498e-05" />
-    </inertial>
-  </link>
+      <inertia ixx="3.3055381e-04" ixy="-9.7940978e-08" ixz="-3.8505711e-05" iyy="3.4290447e-04" iyz="-1.5717516e-06" izz="6.0346498e-05" />
+    </inertial>
+  </link> -->
   <!--  Joint 3 -->
-  <joint name="joint3" type="revolute">
+  <!-- <joint name="joint3" type="revolute">
     <parent link="link3"/>
     <child link="link4"/>
@@ -133,30 +128,28 @@
     <axis xyz="0 1 0"/>
     <limit velocity="4.8" effort="1" lower="-0.94247779607" upper="1.38230076758" />
-  </joint>
+  </joint> -->
   <!--  Link 4 -->
-  <link name="link4">
-    <visual>
-      <origin xyz="0 0 0" rpy="0 0 0"/>
-      <geometry>
-        <mesh filename="package://open_manipulator_x_description/meshes/chain_link4.stl" scale="0.001 0.001 0.001"/>
-      </geometry>
-      <material name="grey"/>
-    </visual>
-    <collision>
-      <origin xyz="0 0 0" rpy="0 0 0"/>
-      <geometry>
-        <mesh filename="package://open_manipulator_x_description/meshes/chain_link4.stl" scale="0.001 0.001 0.001"/>
-      </geometry>
-    </collision>
-     <inertial>
+  <!-- <link name="link4">
+    <visual>
+      <origin xyz="0 0 0" rpy="0 0 0"/>
+      <geometry>
+        <mesh filename="file://$(find open_manipulator_x_description)/meshes/chain_link4.stl" scale="0.001 0.001 0.001"/>
+      </geometry>
+      <material name="grey"/>
+    </visual>
+    <collision>
+      <origin xyz="0 0 0" rpy="0 0 0"/>
+      <geometry>
+        <mesh filename="file://$(find open_manipulator_x_description)/meshes/chain_link4.stl" scale="0.001 0.001 0.001"/>
+      </geometry>
+    </collision>
+    <inertial>
       <origin xyz="9.0909590e-02 3.8929816e-04 2.2413279e-04" />
       <mass value="1.3274562e-01" />
-      <inertia ixx="3.0654178e-05" ixy="-1.2764155e-06" ixz="-2.6874417e-07"
-               iyy="2.4230292e-04" iyz="1.1559550e-08"
-               izz="2.5155057e-04" />
-    </inertial>
-  </link>
+      <inertia ixx="3.0654178e-05" ixy="-1.2764155e-06" ixz="-2.6874417e-07" iyy="2.4230292e-04" iyz="1.1559550e-08" izz="2.5155057e-04" />
+    </inertial>
+  </link> -->
   <!--  Joint 4 -->
-  <joint name="joint4" type="revolute">
+  <!-- <joint name="joint4" type="revolute">
     <parent link="link4"/>
     <child link="link5"/>
@@ -164,30 +157,28 @@
     <axis xyz="0 1 0"/>
     <limit velocity="4.8" effort="1" lower="-1.79070781255" upper="2.04203522483" />
-  </joint>
+  </joint> -->
   <!--  Link 5 -->
-  <link name="link5">
-    <visual>
-      <origin xyz="0 0 0" rpy="0 0 0"/>
-      <geometry>
-        <mesh filename="package://open_manipulator_x_description/meshes/chain_link5.stl" scale="0.001 0.001 0.001"/>
-      </geometry>
-      <material name="grey"/>
-    </visual>
-    <collision>
-      <origin xyz="0 0 0" rpy="0 0 0"/>
-      <geometry>
-        <mesh filename="package://open_manipulator_x_description/meshes/chain_link5.stl" scale="0.001 0.001 0.001"/>
-      </geometry>
-    </collision>
-     <inertial>
+  <!-- <link name="link5">
+    <visual>
+      <origin xyz="0 0 0" rpy="0 0 0"/>
+      <geometry>
+        <mesh filename="file://$(find open_manipulator_x_description)/meshes/chain_link5.stl" scale="0.001 0.001 0.001"/>
+      </geometry>
+      <material name="grey"/>
+    </visual>
+    <collision>
+      <origin xyz="0 0 0" rpy="0 0 0"/>
+      <geometry>
+        <mesh filename="file://$(find open_manipulator_x_description)/meshes/chain_link5.stl" scale="0.001 0.001 0.001"/>
+      </geometry>
+    </collision>
+    <inertial>
       <origin xyz="4.4206755e-02 3.6839985e-07 8.9142216e-03" />
       <mass value="1.4327573e-01" />
-      <inertia ixx="8.0870749e-05" ixy="0.0" ixz="-1.0157896e-06"
-               iyy="7.5980465e-05" iyz="0.0"
-               izz="9.3127351e-05" />
-    </inertial>
-  </link>
+      <inertia ixx="8.0870749e-05" ixy="0.0" ixz="-1.0157896e-06" iyy="7.5980465e-05" iyz="0.0" izz="9.3127351e-05" />
+    </inertial>
+  </link> -->
   <!--  Gripper joint -->
-  <joint name="gripper" type="prismatic">
+  <!-- <joint name="gripper" type="prismatic">
     <parent link="link5"/>
     <child link="gripper_link"/>
@@ -195,11 +186,11 @@
     <axis xyz="0 1 0"/>
     <limit velocity="4.8" effort="1" lower="-0.010" upper="0.019" />
-  </joint>
+  </joint> -->
   <!--  Gripper link -->
-  <link name="gripper_link">
+  <!-- <link name="gripper_link">
     <visual>
       <origin xyz="0.0 0.0 0" rpy="0 0 0"/>
       <geometry>
-        <mesh filename="package://open_manipulator_x_description/meshes/chain_link_grip_l.stl" scale="0.001 0.001 0.001"/>
+        <mesh filename="file://$(find open_manipulator_x_description)/meshes/chain_link_grip_l.stl" scale="0.001 0.001 0.001"/>
       </geometry>
       <material name="grey"/>
@@ -208,5 +199,5 @@
       <origin xyz="0.0 0.0 0" rpy="0 0 0"/>
       <geometry>
-        <mesh filename="package://open_manipulator_x_description/meshes/chain_link_grip_l.stl" scale="0.001 0.001 0.001"/>
+        <mesh filename="file://$(find open_manipulator_x_description)/meshes/chain_link_grip_l.stl" scale="0.001 0.001 0.001"/>
       </geometry>
     </collision>
@@ -214,11 +205,9 @@
       <origin xyz="0 0 0" />
       <mass value="1.0e-03" />
-      <inertia ixx="1.0e-03" ixy="0.0" ixz="0.0"
-               iyy="1.0e-03" iyz="0.0"
-               izz="1.0e-03" />
-    </inertial>
-  </link>
+      <inertia ixx="1.0e-03" ixy="0.0" ixz="0.0" iyy="1.0e-03" iyz="0.0" izz="1.0e-03" />
+    </inertial>
+  </link> -->
   <!--  Gripper joint sub -->
-  <joint name="gripper_sub" type="prismatic">
+  <!-- <joint name="gripper_sub" type="prismatic">
     <parent link="link5"/>
     <child link="gripper_link_sub"/>
@@ -227,11 +216,11 @@
     <limit velocity="4.8" effort="1" lower="-0.010" upper="0.019" />
     <mimic joint="gripper" multiplier="1"/>
-  </joint>
+  </joint> -->
   <!--  Gripper link sub -->
-  <link name="gripper_link_sub">
+  <!-- <link name="gripper_link_sub">
     <visual>
       <origin xyz="0.0 -0.0 0" rpy="0 0 0"/>
       <geometry>
-        <mesh filename="package://open_manipulator_x_description/meshes/chain_link_grip_r.stl" scale="0.001 0.001 0.001"/>
+        <mesh filename="file://$(find open_manipulator_x_description)/meshes/chain_link_grip_r.stl" scale="0.001 0.001 0.001"/>
       </geometry>
       <material name="grey"/>
@@ -240,5 +229,5 @@
       <origin xyz="0.0 -0.0 0" rpy="0 0 0"/>
       <geometry>
-        <mesh filename="package://open_manipulator_x_description/meshes/chain_link_grip_r.stl" scale="0.001 0.001 0.001"/>
+        <mesh filename="file://$(find open_manipulator_x_description)/meshes/chain_link_grip_r.stl" scale="0.001 0.001 0.001"/>
       </geometry>
     </collision>
@@ -246,17 +235,15 @@
       <origin xyz="0 0 0" />
       <mass value="1.0e-03" />
-      <inertia ixx="1.0e-03" ixy="0.0" ixz="0.0"
-               iyy="1.0e-03" iyz="0.0"
-               izz="1.0e-03" />
-    </inertial>
-  </link>
+      <inertia ixx="1.0e-03" ixy="0.0" ixz="0.0" iyy="1.0e-03" iyz="0.0" izz="1.0e-03" />
+    </inertial>
+  </link> -->
   <!-- end effector joint -->
-  <joint name="end_effector_joint" type="fixed">
+  <!-- <joint name="end_effector_joint" type="fixed">
     <origin xyz="0.126 0.0 0.0" rpy="0 0 0"/>
     <parent link="link5"/>
     <child link="end_effector_link"/>
-  </joint>
+  </joint> -->
   <!-- end effector link -->
-  <link name="end_effector_link">
+  <!-- <link name="end_effector_link">
     <visual>
       <origin xyz="0 0 0" rpy="0 0 0"/>
@@ -265,15 +252,13 @@
       </geometry>
       <material name="red"/>
-     </visual>
+    </visual>
     <inertial>
       <origin xyz="0 0 0" />
       <mass value="1.0e-03" />
-      <inertia ixx="1.0e-03" ixy="0.0" ixz="0.0"
-               iyy="1.0e-03" iyz="0.0"
-               izz="1.0e-03" />
-    </inertial>
-  </link>
+      <inertia ixx="1.0e-03" ixy="0.0" ixz="0.0" iyy="1.0e-03" iyz="0.0" izz="1.0e-03" />
+    </inertial>
+  </link> -->
   <!-- Realsense Camera Joint Position -->
-  <joint name="camera_joint" type="fixed">
+  <!-- <joint name="camera_joint" type="fixed">
     <axis xyz="0 1 0" />
     <origin xyz="0.070 0.032 0.052" rpy="0 0 0"/>
@@ -281,4 +266,4 @@
     <child link="camera_link"/>
   </joint>
-  <link name="camera_link"/>
+  <link name="camera_link"/> -->
 </robot>
