Commit message: fix: urdf controllers

File: open_manipulator_x_description/urdf/open_manipulator_x.gazebo.xacro (robot description, xacro)
@@ -34,58 +34,53 @@
   </gazebo>
   <!-- ros_control plugin -->
+  <ros2_control name="GazeboSystem" type="system">
+    <hardware>
+      <plugin>gazebo_ros2_control/GazeboSystem</plugin>
+    </hardware>
+    <joint name="joint1">
+      <command_interface name="position">
+        <param name="min">-2.356</param>
+        <param name="max">5.934</param>
+      </command_interface>
+      <state_interface name="position" />
+      <state_interface name="velocity" />
+    </joint>
+    <joint name="joint2">
+      <command_interface name="position">
+        <param name="min">${-pi*0.57}</param>
+        <param name="max">${pi*0.5}</param>
+      </command_interface>
+      <state_interface name="position" />
+      <state_interface name="velocity" />
+    </joint>
+    <joint name="joint3">
+      <command_interface name="position">
+        <param name="min">${-pi*0.3}</param>
+        <param name="max">${pi*0.44}</param>
+      </command_interface>
+      <state_interface name="position" />
+      <state_interface name="velocity" />
+    </joint>
+    <joint name="joint4">
+      <command_interface name="position">
+        <param name="min">${-pi*0.57}</param>
+        <param name="max">${pi*0.65}</param>
+      </command_interface>
+      <state_interface name="position" />
+      <state_interface name="velocity" />
+    </joint>
+    <joint name="gripper">
+      <command_interface name="position">
+        <param name="min">-0.010</param>
+        <param name="max">0.019</param>
+      </command_interface>
+      <state_interface name="position" />
+      <state_interface name="velocity" />
+    </joint>
+  </ros2_control>
   <gazebo>
-    <plugin name="gazebo_ros_control" filename="libgazebo_ros_control.so">
-      <controlPeriod>0.001</controlPeriod>
-      <robotSimType>gazebo_ros_control/DefaultRobotHWSim</robotSimType>
+    <plugin name="gazebo_ros2_control" filename="libgazebo_ros2_control.so">
+      <parameters>$(find open_manipulator_x_moveit_config)/config/ros2_controllers.yaml</parameters>
     </plugin>
   </gazebo>
-  <!-- loading plugin: mimic joints works in gazebo now -->
-  <!-- <gazebo>
-    <plugin name="gazebo_gripper_ros_control" filename="libroboticsgroup_gazebo_mimic_joint_plugin.so">
-      <joint>gripper</joint>
-      <mimicJoint>gripper_sub</mimicJoint>
-      <multiplier>1.0</multiplier>
-      <offset>0.0</offset>
-    </plugin>
-  </gazebo> -->
-  <!-- camera -->
-  <!-- Noise is sampled independently per pixel on each frame.
-        That pixel's noise value is added to each of its color
-        channels, which at that point lie in the range [0,1]. -->
-  <!-- <gazebo reference="camera_link">
-    <sensor type="camera" name="intel_realsense_r200">
-      <update_rate>30.0</update_rate>
-      <camera name="head">
-        <horizontal_fov>1.02974</horizontal_fov>
-        <image>
-          <width>1920</width>
-          <height>1080</height>
-          <format>R8G8B8</format>
-        </image>
-        <clip>
-          <near>0.02</near>
-          <far>300</far>
-        </clip>
-        <noise>
-          <type>gaussian</type>
-          <mean>0.0</mean>
-          <stddev>0.007</stddev>
-        </noise>
-      </camera>
-      <plugin name="camera_controller" filename="libgazebo_ros_camera.so">
-        <alwaysOn>true</alwaysOn>
-        <updateRate>0.0</updateRate>
-        <cameraName>camera/color</cameraName>
-        <imageTopicName>image_raw</imageTopicName>
-        <cameraInfoTopicName>camera_info</cameraInfoTopicName>
-        <frameName>camera_link</frameName>
-        <hackBaseline>0.07</hackBaseline>
-        <distortionK1>0.0</distortionK1>
-        <distortionK2>0.0</distortionK2>
-        <distortionK3>0.0</distortionK3>
-        <distortionT1>0.0</distortionT1>
-        <distortionT2>0.0</distortionT2>
-      </plugin>
-    </sensor>
-  </gazebo> -->
 </robot>

File: open_manipulator_x_description/urdf/open_manipulator_x_robot.urdf.xacro (robot description, xacro)
@@ -10,5 +10,5 @@
   </xacro:if>
   <!-- Import Transmission -->
-  <xacro:include filename="$(find open_manipulator_x_description)/urdf/open_manipulator_x.transmission.xacro" />
+  <!-- <xacro:include filename="$(find open_manipulator_x_description)/urdf/open_manipulator_x.transmission.xacro" /> -->
   <!-- Import URDF -->
   <xacro:include filename="$(find open_manipulator_x_description)/urdf/open_manipulator_x.urdf.xacro" />

Commit message: fix: mimic gripper plugin

File: open_manipulator_x_description/urdf/open_manipulator_x.gazebo.xacro (robot description, xacro)
@@ -80,4 +80,11 @@
   </ros2_control>
   <gazebo>
+    <plugin filename="libroboticsgroup_upatras_gazebo_mimic_joint_plugin.so" name="mimic_joint">
+      <joint>gripper</joint>
+      <mimicJoint>gripper_sub</mimicJoint>
+      <multiplier>1.0</multiplier>
+      <offset>0.0</offset>
+      <maxEffort>5.0</maxEffort>
+    </plugin>
     <plugin name="gazebo_ros2_control" filename="libgazebo_ros2_control.so">
       <parameters>$(find open_manipulator_x_moveit_config)/config/ros2_controllers.yaml</parameters>

Commit message: fix: urdf collision

File: open_manipulator_x_description/urdf/open_manipulator_x.gazebo.xacro (robot description, xacro)
@@ -78,4 +78,12 @@
       <state_interface name="velocity" />
     </joint>
+    <joint name="gripper_sub">
+      <command_interface name="position">
+        <param name="min">-0.010</param>
+        <param name="max">0.019</param>
+      </command_interface>
+      <state_interface name="position" />
+      <state_interface name="velocity" />
+    </joint>
   </ros2_control>
   <gazebo>

File: open_manipulator_x_description/urdf/open_manipulator_x.urdf.xacro (robot description, xacro)
@@ -212,5 +212,5 @@
   <!-- end effector link -->
   <link name="end_effector_link">
-    <visual>
+    <!-- <visual>
       <origin xyz="0 0 0" rpy="0 0 0"/>
       <geometry>
@@ -223,5 +223,5 @@
       <mass value="1.0e-03" />
       <inertia ixx="1.0e-03" ixy="0.0" ixz="0.0" iyy="1.0e-03" iyz="0.0" izz="1.0e-03" />
-    </inertial>
+    </inertial> -->
   </link>
   <!-- Realsense Camera Joint Position -->
